File: pcb-1/pcb-1.kicad_sch (KiCad schematic)
At the start: 8 parts, among them J1 Raspberry_Pi_2_3, J2 Screw_Terminal_01x03, J3 Conn_01x07_Socket, J4 Screw_Terminal_01x02, J5 Conn_01x02_Socket, U1 Pico, U2 TSR 2-2450

Commit message: Added title to board
Other:
- title: (none) -> Power Distribution Board
Changed lines of the file:
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@@
 (kicad_sch (version 20230121) (generator eeschema)
   (paper "A4")
+  (title_block
+    (title "Power Distribution Board")
+    (rev "1")
+  )
   (junction (at 54.61 83.82) (diameter 0) (color 0 0 0 0)
   )
@@
     )
     (pin "1")
+    (pin "2")
     (pin "3")
+    (instances
+      (project "pcb-1"
+        (path "/43486df0-1e41-4516-8027-8058a2e1c66f"
+          (reference "U2") (unit 1)
+        )
+      )
+    )
+  )
+  (symbol (lib_id "power:+5V") (at 104.14 66.04 0) (unit 1)
+    (in_bom yes) (on_board yes) (dnp no) (fields_autoplaced)
+    (property "Reference" "#PWR02" (at 104.14 69.85 0)
+      (effects (font (size 1.27 1.27)) hide)
+    )
+    (property "Value" "+5V" (at 104.14 60.96 0)
+      (effects (font (size 1.27 1.27)))
+    )
+    (property "Footprint" "" (at 104.14 66.04 0)
+      (effects (font (size 1.27 1.27)) hide)
+    )
+    (property "Datasheet" "" (at 104.14 66.04 0)
+      (effects (font (size 1.27 1.27)) hide)
+    )
+    (pin "1")
+    (instances
+      (project "pcb-1"
+        (path "/43486df0-1e41-4516-8027-8058a2e1c66f"
+          (reference "#PWR02") (unit 1)
+        )
+      )
+    )
+  )
+  (symbol (lib_id "Connector:Raspberry_Pi_2_3") (at 162.56 90.17 0) (unit 1)
+    (in_bom yes) (on_board yes) (dnp no) (fields_autoplaced)
+    (property "Reference" "J1" (at 169.8341 54.61 0)
+      (effects (font (size 1.27 1.27)) (justify left))
+    )
+    (property "Value" "Raspberry_Pi_2_3" (at 169.8341 57.15 0)
+      (effects (font (size 1.27 1.27)) (justify left))
+    )
+    (property "Footprint" "pi:raspberrypi_2_3" (at 162.56 90.17 0)
+      (effects (font (size 1.27 1.27)) hide)
+    )
+    (property "Datasheet" "https://www.raspberrypi.org/documentation/hardware/raspberrypi/schematics/rpi_SCH_3bplus_1p0_reduced.pdf" (at 162.56 90.17 0)
+      (effects (font (size 1.27 1.27)) hide)
+    )
+    (pin "1")
+    (pin "10")
+    (pin "11")
+    (pin "12")
+    (pin "13")
+    (pin "14")
+    (pin "15")
+    (pin "16")
+    (pin "17")
+    (pin "18")
+    (pin "19")
     (pin "2")
-    (instances
-      (project "pcb-1"
-        (path "/43486df0-1e41-4516-8027-8058a2e1c66f"
-          (reference "U2") (unit 1)
-        )
-      )
-    )
-  )
-  (symbol (lib_id "power:+5V") (at 104.14 66.04 0) (unit 1)
-    (in_bom yes) (on_board yes) (dnp no) (fields_autoplaced)
-    (property "Reference" "#PWR02" (at 104.14 69.85 0)
-      (effects (font (size 1.27 1.27)) hide)
-    )
-    (property "Value" "+5V" (at 104.14 60.96 0)
-      (effects (font (size 1.27 1.27)))
-    )
-    (property "Footprint" "" (at 104.14 66.04 0)
-      (effects (font (size 1.27 1.27)) hide)
-    )
-    (property "Datasheet" "" (at 104.14 66.04 0)
-      (effects (font (size 1.27 1.27)) hide)
-    )
-    (pin "1")
-    (instances
-      (project "pcb-1"
-        (path "/43486df0-1e41-4516-8027-8058a2e1c66f"
-          (reference "#PWR02") (unit 1)
-        )
-      )
-    )
-  )
-  (symbol (lib_id "Connector:Raspberry_Pi_2_3") (at 162.56 90.17 0) (unit 1)
-    (in_bom yes) (on_board yes) (dnp no) (fields_autoplaced)
-    (property "Reference" "J1" (at 169.8341 54.61 0)
-      (effects (font (size 1.27 1.27)) (justify left))
-    )
-    (property "Value" "Raspberry_Pi_2_3" (at 169.8341 57.15 0)
-      (effects (font (size 1.27 1.27)) (justify left))
-    )
-    (property "Footprint" "pi:raspberrypi_2_3" (at 162.56 90.17 0)
-      (effects (font (size 1.27 1.27)) hide)
-    )
-    (property "Datasheet" "https://www.raspberrypi.org/documentation/hardware/raspberrypi/schematics/rpi_SCH_3bplus_1p0_reduced.pdf" (at 162.56 90.17 0)
-      (effects (font (size 1.27 1.27)) hide)
-    )
+    (pin "20")
+    (pin "21")
+    (pin "22")
+    (pin "23")
+    (pin "24")
+    (pin "25")
+    (pin "26")
+    (pin "27")
+    (pin "28")
+    (pin "29")
+    (pin "3")
+    (pin "30")
+    (pin "31")
+    (pin "32")
+    (pin "33")
     (pin "34")
     (pin "35")
-    (pin "31")
+    (pin "36")
+    (pin "37")
+    (pin "38")
+    (pin "39")
+    (pin "4")
+    (pin "40")
     (pin "5")
     (pin "6")
-    (pin "25")
-    (pin "18")
-    (pin "3")
-    (pin "17")
+    (pin "7")
     (pin "8")
-    (pin "26")
-    (pin "30")
-    (pin "27")
-    (pin "33")
-    (pin "22")
-    (pin "21")
-    (pin "32")
-    (pin "7")
-    (pin "20")
     (pin "9")
-    (pin "39")
-    (pin "23")
-    (pin "28")
-    (pin "2")
-    (pin "24")
-    (pin "19")
-    (pin "15")
-    (pin "14")
-    (pin "13")
-    (pin "12")
-    (pin "11")
-    (pin "10")
-    (pin "1")
-    (pin "29")
-    (pin "16")
-    (pin "36")
-    (pin "40")
-    (pin "37")
-    (pin "38")
-    (pin "4")
     (instances
       (project "pcb-1"
@@
       (effects (font (size 1.27 1.27)) hide)
     )
+    (pin "1")
+    (pin "2")
     (pin "3")
-    (pin "1")
-    (pin "2")
     (instances
       (project "pcb-1"
@@
     )
     (pin "1")
-    (pin "21")
-    (pin "16")
-    (pin "9")
-    (pin "36")
-    (pin "41")
-    (pin "20")
-    (pin "26")
+    (pin "10")
     (pin "11")
     (pin "12")
+    (pin "13")
+    (pin "14")
+    (pin "15")
+    (pin "16")
+    (pin "17")
+    (pin "18")
+    (pin "19")
+    (pin "2")
+    (pin "20")
+    (pin "21")
     (pin "22")
-    (pin "14")
-    (pin "5")
-    (pin "15")
-    (pin "38")
-    (pin "35")
-    (pin "33")
+    (pin "23")
+    (pin "24")
+    (pin "25")
+    (pin "26")
+    (pin "27")
     (pin "28")
     (pin "29")
-    (pin "27")
-    (pin "17")
+    (pin "3")
+    (pin "30")
     (pin "31")
+    (pin "32")
+    (pin "33")
+    (pin "34")
+    (pin "35")
+    (pin "36")
+    (pin "37")
+    (pin "38")
+    (pin "39")
+    (pin "4")
+    (pin "40")
+    (pin "41")
+    (pin "42")
     (pin "43")
-    (pin "18")
-    (pin "4")
-    (pin "30")
-    (pin "25")
-    (pin "34")
-    (pin "42")
-    (pin "24")
-    (pin "19")
-    (pin "39")
-    (pin "32")
-    (pin "23")
-    (pin "10")
-    (pin "37")
-    (pin "2")
-    (pin "3")
-    (pin "8")
-    (pin "13")
-    (pin "40")
+    (pin "5")
     (pin "6")
     (pin "7")
+    (pin "8")
+    (pin "9")
     (instances
       (project "pcb-1"
@@
     )
     (pin "1")
+    (pin "2")
+    (pin "3")
+    (pin "4")
     (pin "5")
-    (pin "3")
+    (pin "6")
     (pin "7")
+    (instances
+      (project "pcb-1"
+        (path "/43486df0-1e41-4516-8027-8058a2e1c66f"
+          (reference "J3") (unit 1)
+        )
+      )
+    )
+  )
+  (symbol (lib_id "power:+5V") (at 52.07 177.8 0) (unit 1)
+    (in_bom yes) (on_board yes) (dnp no) (fields_autoplaced)
+    (property "Reference" "#PWR01" (at 52.07 181.61 0)
+      (effects (font (size 1.27 1.27)) hide)
+    )
+    (property "Value" "+5V" (at 52.07 172.72 0)
+      (effects (font (size 1.27 1.27)))
+    )
+    (property "Footprint" "" (at 52.07 177.8 0)
+      (effects (font (size 1.27 1.27)) hide)
+    )
+    (property "Datasheet" "" (at 52.07 177.8 0)
+      (effects (font (size 1.27 1.27)) hide)
+    )
+    (pin "1")
+    (instances
+      (project "pcb-1"
+        (path "/43486df0-1e41-4516-8027-8058a2e1c66f"
+          (reference "#PWR01") (unit 1)
+        )
+      )
+    )
+  )
+  (symbol (lib_id "Connector:Conn_01x02_Socket") (at 215.9 154.94 0) (unit 1)
+    (in_bom yes) (on_board yes) (dnp no) (fields_autoplaced)
+    (property "Reference" "J5" (at 217.17 154.94 0)
+      (effects (font (size 1.27 1.27)) (justify left))
+    )
+    (property "Value" "Conn_01x02_Socket" (at 217.17 157.48 0)
+      (effects (font (size 1.27 1.27)) (justify left))
+    )
+    (property "Footprint" "Connector_AMASS:AMASS_XT60-F_1x02_P7.20mm_Vertical" (at 215.9 154.94 0)
+      (effects (font (size 1.27 1.27)) hide)
+    )
+    (property "Datasheet" "~" (at 215.9 154.94 0)
+      (effects (font (size 1.27 1.27)) hide)
+    )
+    (pin "1")
     (pin "2")
-    (pin "6")
-    (pin "4")
-    (instances
-      (project "pcb-1"
-        (path "/43486df0-1e41-4516-8027-8058a2e1c66f"
-          (reference "J3") (unit 1)
-        )
-      )
-    )
-  )
-  (symbol (lib_id "power:+5V") (at 52.07 177.8 0) (unit 1)
-    (in_bom yes) (on_board yes) (dnp no) (fields_autoplaced)
-    (property "Reference" "#PWR01" (at 52.07 181.61 0)
-      (effects (font (size 1.27 1.27)) hide)
-    )
-    (property "Value" "+5V" (at 52.07 172.72 0)
-      (effects (font (size 1.27 1.27)))
-    )
-    (property "Footprint" "" (at 52.07 177.8 0)
-      (effects (font (size 1.27 1.27)) hide)
-    )
-    (property "Datasheet" "" (at 52.07 177.8 0)
-      (effects (font (size 1.27 1.27)) hide)
-    )
-    (pin "1")
-    (instances
-      (project "pcb-1"
-        (path "/43486df0-1e41-4516-8027-8058a2e1c66f"
-          (reference "#PWR01") (unit 1)
-        )
-      )
-    )
-  )
-  (symbol (lib_id "Connector:Conn_01x02_Socket") (at 215.9 154.94 0) (unit 1)
-    (in_bom yes) (on_board yes) (dnp no) (fields_autoplaced)
-    (property "Reference" "J5" (at 217.17 154.94 0)
-      (effects (font (size 1.27 1.27)) (justify left))
-    )
-    (property "Value" "Conn_01x02_Socket" (at 217.17 157.48 0)
-      (effects (font (size 1.27 1.27)) (justify left))
-    )
-    (property "Footprint" "Connector_AMASS:AMASS_XT60-F_1x02_P7.20mm_Vertical" (at 215.9 154.94 0)
-      (effects (font (size 1.27 1.27)) hide)
-    )
-    (property "Datasheet" "~" (at 215.9 154.94 0)
-      (effects (font (size 1.27 1.27)) hide)
-    )
-    (pin "2")
-    (pin "1")
-    (instances
-      (project "pcb-1"
+    (instances
+      (project "pcb-1"

Commit message: Added pi code
Other:
- note added: "Raspberry Pi"
- note added: "Raspberry Pi Pico"
- note added: "TSR"
- note removed: "TODO: POWER DELIVERY"
Changed lines of the file:
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@@
     (stroke (width 0) (type default))
   )
-  (text "TODO: POWER DELIVERY\n" (at 219.71 107.95 0)
+  (text "Raspberry Pi" (at 148.59 43.18 0)
+    (effects (font (size 3 3)) (justify left bottom))
+  )
+  (text "TSR" (at 229.235 112.395 0)
     (effects (font (size 3 3)) (justify left bottom))
   )
@@
     (effects (font (size 4 4)) (justify left bottom))
   )
+  (text "Raspberry Pi Pico" (at 60.325 53.975 0)
+    (effects (font (size 3 3)) (justify left bottom))
+  )
   (text "SERVO\n\n" (at 97.79 161.29 0)
