File: pcb-v2/pcb-v2.kicad_pcb (KiCad board)
At the start: 2 copper layers, 31.8 x 57.9 mm, 5 parts, among them J1 Conn_02x20_Odd_Even, J2 Conn_01x07_Socket, J3 Screw_Terminal_01x03, J4 Screw_Terminal_01x02

Commit message: pcb-v2 r2
Other:
- board text added: "+3.3v"
- board text added: "+5V"
- board text added: "+5v"
- board text added: "ESC"
- board text added: "GND"
- board text added: "SCL"
- board text added: "SDA"
- board text added: "SERVO"
Changed lines of the file:
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@@
   (gr_line (start 181.76875 80.16875) (end 182.5625 80.16875)
     (stroke (width 0.1) (type default)) (layer "Edge.Cuts"))
+  (gr_text "SDA" (at 192.88125 94.45625) (layer "F.SilkS")
+    (effects (font (size 1.5 1.5) (thickness 0.3) bold) (justify left bottom))
+  )
+  (gr_text "SCL" (at 192.88125 96.8375) (layer "F.SilkS")
+    (effects (font (size 1.5 1.5) (thickness 0.3) bold) (justify left bottom))
+  )
+  (gr_text "ESC" (at 193.675 115.8875) (layer "F.SilkS")
+    (effects (font (size 1.5 1.5) (thickness 0.3) bold) (justify left bottom))
+  )
+  (gr_text "GND" (at 192.88125 99.21875) (layer "F.SilkS")
+    (effects (font (size 1.5 1.5) (thickness 0.3) bold) (justify left bottom))
+  )
+  (gr_text "GND\n" (at 193.675 127.79375) (layer "F.SilkS")
+    (effects (font (size 1.5 1.5) (thickness 0.3) bold) (justify left bottom))
+  )
+  (gr_text "+3.3v" (at 199.23125 85.725) (layer "F.SilkS")
+    (effects (font (size 1.5 1.5) (thickness 0.3) bold) (justify left bottom))
+  )
+  (gr_text "GND" (at 193.675 111.125) (layer "F.SilkS")
+    (effects (font (size 1.5 1.5) (thickness 0.3) bold) (justify left bottom))
+  )
+  (gr_text "+5v" (at 207.9625 83.34375) (layer "F.SilkS")
+    (effects (font (size 1.5 1.5) (thickness 0.3) bold) (justify left bottom))
+  )
+  (gr_text "+5V" (at 192.88125 134.14375) (layer "F.SilkS")
+    (effects (font (size 1.5 1.5) (thickness 0.3) bold) (justify left bottom))
+  )
+  (gr_text "+5V" (at 192.88125 101.6) (layer "F.SilkS")
+    (effects (font (size 1.5 1.5) (thickness 0.3) bold) (justify left bottom))
+  )
+  (gr_text "SERVO\n" (at 193.675 123.03125) (layer "F.SilkS")
+    (effects (font (size 1.5 1.5) (thickness 0.3) bold) (justify left bottom))
+  )
   (segment (start 186.825 132.482601) (end 193.770966 132.482601) (width 1.2) (layer "F.Cu") (net 1))
   (segment (start 186.617601 100.892601) (end 186.53125 100.80625) (width 1.2) (layer "F.Cu") (net 1))

Commit message: pcb-v2 rc1
Parts:
- J1: footprint Connector_PinHeader_2.54mm:PinHeader_2x20_P2.54mm_Vertical -> Connector_PinSocket_2.54mm:PinSocket_2x20_P2.54mm_Vertical; moved to B.Cu
- J3: footprint terminal:CONN_1935174_PXC -> Connector_PinHeader_2.54mm:PinHeader_1x03_P2.54mm_Horizontal
- J4: footprint terminal:CONN2_710002_WRE -> Connector_PinHeader_2.54mm:PinHeader_1x02_P2.54mm_Horizontal
- moved J4 1.09 mm to (186.5, 115.1), turned to 180 degrees
- moved J3 0.29 mm to (186.5, 132.5), turned to 180 degrees
- turned J1 to 180 degrees
Routing:
- net SDA: track 23.5 -> 20.3 mm, vias 2 -> 0
- net SCL: track 23.1 -> 20.3 mm, vias 2 -> 0
- net SERVO: track 52.4 -> 54.9 mm
- net +5V: track 100.5 -> 102.9 mm, vias 5 -> 4
- net ESC: track 30.5 -> 31.1 mm
Other:
- board size 31.8 x 57.9 mm -> 31 x 57.9 mm
- board text added: "ESC/33"
