File: pcb-v2/pcb-v2.kicad_sch (KiCad schematic)
At the start: 1 part, among them J1 Conn_02x20_Odd_Even

Commit message: pcb-v2 r1
Parts:
- added C1: 100uf, Capacitor_THT:CP_Radial_Tantal_D10.5mm_P5.00mm, symbol Device:C
- added J2: Conn_01x07_Socket, Connector_PinHeader_2.54mm:PinHeader_1x07_P2.54mm_Vertical, symbol Connector:Conn_01x07_Socket
- added J3: Screw_Terminal_01x03, terminal:CONN_1935174_PXC, symbol Connector:Screw_Terminal_01x03
- added J4: Screw_Terminal_01x02, terminal:CONN2_710002_WRE, symbol Connector:Screw_Terminal_01x02
- J1: footprint Connector_PinHeader_1.00mm:PinHeader_2x20_P1.00mm_Vertical -> Connector_PinHeader_2.54mm:PinHeader_2x20_P2.54mm_Vertical
Connections:
- net +5V: now also C1.1, J2.7 (Pin_7), J3.1 (Pin_1)
- net GND: now also C1.2, J2.3 (Pin_3), J2.6 (Pin_6), J3.2 (Pin_2), J4.2 (Pin_2)
- net SDA: now reaches J1.3 (Pin_3)
- net SDA: now also J2.4 (Pin_4)
- net SERVO: now reaches J1.32 (Pin_32)
- net SERVO: now also J3.3 (Pin_3)
- net ESC: now reaches J1.33 (Pin_33)
- net ESC: now also J4.1 (Pin_1)
- net SCL: now reaches J1.5 (Pin_5)
- net SCL: now also J2.5 (Pin_5)
- no-connect marks 0 -> 26
Other:
- note added: "BMX"
- note added: "ESC"
- note added: "SERVO"

Commit message: pcb-v2 rc1
Parts:
- J1: footprint Connector_PinHeader_2.54mm:PinHeader_2x20_P2.54mm_Vertical -> Connector_PinSocket_2.54mm:PinSocket_2x20_P2.54mm_Vertical
- J3: footprint terminal:CONN_1935174_PXC -> Connector_PinHeader_2.54mm:PinHeader_1x03_P2.54mm_Horizontal
- J4: footprint terminal:CONN2_710002_WRE -> Connector_PinHeader_2.54mm:PinHeader_1x02_P2.54mm_Horizontal
Changed lines of the file:
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@@
       (effects (font (size 1.27 1.27)))
     )
-    (property "Footprint" "Connector_PinHeader_2.54mm:PinHeader_2x20_P2.54mm_Vertical" (at 114.3 77.47 0)
-      (effects (font (size 1.27 1.27)) hide)
+    (property "Footprint" "Connector_PinSocket_2.54mm:PinSocket_2x20_P2.54mm_Vertical" (at 114.3 77.47 0)
+      (effects (font (size 1.27 1.27)))
     )
     (property "Datasheet" "~" (at 114.3 77.47 0)
@@
       (effects (font (size 1.27 1.27)) (justify left))
     )
-    (property "Footprint" "terminal:CONN2_710002_WRE" (at 166.37 127 0)
+    (property "Footprint" "Connector_PinHeader_2.54mm:PinHeader_1x02_P2.54mm_Horizontal" (at 166.37 127 0)
       (effects (font (size 1.27 1.27)) hide)
     )
@@
       (effects (font (size 1.27 1.27)) (justify left))
     )
-    (property "Footprint" "terminal:CONN_1935174_PXC" (at 123.19 129.54 0)
-      (effects (font (size 1.27 1.27)) hide)
-    )
+    (property "Footprint" "Connector_PinHeader_2.54mm:PinHeader_1x03_P2.54mm_Horizontal" (at 123.19 129.54 0)
+      (effects (font (size 1.27 1.27)) hide)
+    )
